Commit message: Fix top camera visual origin

File: jaime_description/urdf/jaime_asus.urdf.xacro (robot description, xacro)
@@ -241,5 +241,5 @@
       </collision-->
       <visual>
-        <origin xyz="0 0 0" rpy="0 0 0"/>
+        <origin xyz="0 0 0" rpy="${M_PI/2} 0 ${M_PI/2}"/>
         <geometry>
           <!--box size="${camara} ${camara} ${camara}"/-->
