Commit message: added depth camera to sim

File: jaime_description/urdf/jaime.urdf.xacro (robot description, xacro)
@@ -8,4 +8,5 @@
 <robot name="kobuki" xmlns:xacro="http://ros.org/wiki/xacro">
   <xacro:include filename="$(find jaime_description)/urdf/common_properties.urdf.xacro"/>
+  <xacro:include filename="$(find jaime_description)/urdf/jaime_sensors_properties.urdf.xacro"/>
   <xacro:include filename="$(find jaime_description)/urdf/jaime_gazebo.urdf.xacro"/>
   <!-- Kobuki -->
@@ -240,4 +241,91 @@
   </collision>
 </link-->
+<!-- depth camera -->
+    <!-- camera body, with origin at bottom screw mount -->
+    <joint name="camera_joint" type="fixed">
+      <origin xyz="0.0 0.0 0.85" rpy="0 0.610865 0"/>
+      <parent link="base_link"/>
+      <child link="camera_bottom_screw_frame" />
+    </joint>
+    <link name="camera_bottom_screw_frame"/>
+    <joint name="camera_link_joint" type="fixed">
+      <origin xyz="0 ${d435_cam_depth_py} ${d435_cam_depth_pz}" rpy="0 0 0"/>
+      <parent link="camera_bottom_screw_frame"/>
+      <child link="camera_link" />
+    </joint>
+    <link name="camera_link">
+      <visual>
+      <origin xyz="${d435_cam_mount_from_center_offset} ${-d435_cam_depth_py} 0" rpy="${M_PI/2} 0 ${M_PI/2}"/>
+        <geometry>
+          <!-- <box size="${d435_cam_width} ${d435_cam_height} ${d435_cam_depth}"/> -->
+          <mesh filename="package://jaime_description/meshes/d435.dae" />
+          <!--<mesh filename="package://realsense2_description/meshes/d435/d435.dae" />-->
+        </geometry>
+      </visual>
+      <collision>
+        <origin xyz="0 ${-d435_cam_depth_py} 0" rpy="0 0 0"/>
+        <geometry>
+        <box size="${d435_cam_depth} ${d435_cam_width} ${d435_cam_height}"/>
+        </geometry>
+      </collision>
+      <inertial>
+        <!-- The following are not reliable values, and should not be used for modeling -->
+        <mass value="0.564" />
+        <origin xyz="0 0 0" />
+        <inertia ixx="0.003881243" ixy="0.0" ixz="0.0" iyy="0.000498940" iyz="0.0" izz="0.003879257" />
+      </inertial>
+    </link>
+ <!-- camera depth joints and links -->
+  <joint name="camera_depth_joint" type="fixed">
+    <origin xyz="0 0 0" rpy="0 0 0"/>
+    <parent link="camera_link"/>
+    <child link="camera_depth_frame" />
+  </joint>
+  <link name="camera_depth_frame"/>
+  <joint name="camera_depth_optical_joint" type="fixed">
+    <origin xyz="0 0 0" rpy="${-M_PI/2} 0 ${-M_PI/2}" />
+    <parent link="camera_depth_frame" />
+    <child link="camera_depth_optical_frame" />
+  </joint>
+  <link name="camera_depth_optical_frame"/>
+<!-- camera left IR joints and links -->
+<joint name="camera_left_ir_joint" type="fixed">
+  <origin xyz="0 ${d435_cam_depth_to_left_ir_offset} 0" rpy="0 0 0" />
+  <parent link="camera_depth_frame" />
+  <child link="camera_left_ir_frame" />
+</joint>
+<link name="camera_left_ir_frame"/>
+<joint name="camera_left_ir_optical_joint" type="fixed">
+  <origin xyz="0 0 0" rpy="${-M_PI/2} 0 ${-M_PI/2}" />
+  <parent link="camera_left_ir_frame" />
+  <child link="camera_left_ir_optical_frame" />
+</joint>
+<link name="camera_left_ir_optical_frame"/>
+<!-- camera right IR joints and links -->
+<joint name="camera_right_ir_joint" type="fixed">
+  <origin xyz="0 ${d435_cam_depth_to_right_ir_offset} 0" rpy="0 0 0" />
+  <parent link="camera_depth_frame" />
+  <child link="camera_right_ir_frame" />
+</joint>
+<link name="camera_right_ir_frame"/>
+<joint name="camera_right_ir_optical_joint" type="fixed">
+  <origin xyz="0 0 0" rpy="${-M_PI/2} 0 ${-M_PI/2}" />
+  <parent link="camera_right_ir_frame" />
+  <child link="camera_right_ir_optical_frame" />
+</joint>
+<link name="camera_right_ir_optical_frame"/>
+<!-- camera color joints and links -->
+<joint name="camera_color_joint" type="fixed">
+  <origin xyz="0 ${d435_cam_depth_to_color_offset} 0" rpy="0 0 0" />
+  <parent link="camera_depth_frame" />
+  <child link="camera_color_frame" />
+</joint>
+<link name="camera_color_frame"/>
+<joint name="camera_color_optical_joint" type="fixed">
+  <origin xyz="0 0 0" rpy="${-M_PI/2} 0 ${-M_PI/2}" />
+  <parent link="camera_color_frame" />
+  <child link="camera_color_optical_frame" />
+</joint>
+<link name="camera_color_optical_frame"/>
 <!-- Hokuyo Laser -->
 <link name="laser">

File: jaime_description/urdf/jaime_gazebo.urdf.xacro (robot description, xacro)
@@ -1,216 +1,351 @@
 <?xml version="1.0"?>
 <robot name="kobuki_sim" xmlns:xacro="http://ros.org/wiki/xacro">
-  <xacro:macro name="kobuki_sim">
-	  <gazebo reference="wheel_left_link">
-	    <mu1>1.0</mu1>
-	    <mu2>1.0</mu2>
-	    <kp>1000000.0</kp>
-	    <kd>100.0</kd>
-	    <minDepth>0.001</minDepth>
-	    <maxVel>1.0</maxVel>
-	  </gazebo>
-	  <gazebo reference="wheel_right_link">
-	    <mu1>1.0</mu1>
-	    <mu2>1.0</mu2>
-	    <kp>1000000.0</kp>
-	    <kd>100.0</kd>
-	    <minDepth>0.001</minDepth>
-	    <maxVel>1.0</maxVel>
-	  </gazebo>
-	  <gazebo reference="caster_front_link">
-	    <mu1>0.0</mu1>
-	    <mu2>0.0</mu2>
-	    <kp>1000000.0</kp>
-	    <kd>100.0</kd>
-	    <minDepth>0.001</minDepth>
-	    <maxVel>1.0</maxVel>
-	  </gazebo>
-	  <gazebo reference="caster_back_link">
-	    <mu1>0.0</mu1>
-	    <mu2>0.0</mu2>
-	    <kp>1000000.0</kp>
-	    <kd>100.0</kd>
-	    <minDepth>0.001</minDepth>
-	    <maxVel>1.0</maxVel>
-	  </gazebo>
-	  <gazebo reference="base_link">
-	    <mu1>0.3</mu1>
-	    <mu2>0.3</mu2>
-	    <sensor type="contact" name="bumpers">
-	      <always_on>1</always_on>
-	      <update_rate>50.0</update_rate>
-	      <visualize>true</visualize>
-	      <contact>
-	        <collision>base_footprint_fixed_joint_lump__base_collision</collision>
-	      </contact>
-	    </sensor>
-	  </gazebo>
-    <!-- hokuyo -->
-    <gazebo reference="laser">
-      <sensor type="ray" name="head_hokuyo_sensor">
-        <pose>0 0 0.064 0 0 0</pose>
-        <visualize>true</visualize>
-        <update_rate>40</update_rate>
-        <ray>
-          <scan>
-            <horizontal>
-              <samples>1080</samples>
-              <resolution>1</resolution>
-              <min_angle>-1.570796</min_angle>
-              <max_angle>1.570796</max_angle>
-            </horizontal>
-          </scan>
-          <range>
-            <min>0.10</min>
-            <max>4.0</max>
-            <resolution>0.01</resolution>
-          </range>
-          <noise>
-            <type>gaussian</type>
-            <!-- Noise parameters based on published spec for Hokuyo laser
-                 achieving "+-30mm" accuracy at range < 10m.  A mean of 0.0m and
-                 stddev of 0.01m will put 99.7% of samples within 0.03m of the true
-                 reading. -->
-            <mean>0.0</mean>
-            <stddev>0.01</stddev>
-          </noise>
-        </ray>
-        <plugin name="gazebo_ros_head_hokuyo_controller" filename="libgazebo_ros_laser.so">
-          <topicName>scan</topicName>
-          <frameName>laser</frameName>
-        </plugin>
-      </sensor>
-    </gazebo>
-	  <gazebo reference="cliff_sensor_left_link">
-	    <sensor type="ray" name="cliff_sensor_left">
-	      <always_on>true</always_on>
-	      <update_rate>50</update_rate>
-	      <visualize>true</visualize>
-	      <ray>
-	        <scan>
-	          <horizontal>
-	            <samples>50</samples>
-	            <resolution>1.0</resolution>
-	            <min_angle>-0.0436</min_angle>  <!-- -2.5 degree -->
-	            <max_angle>0.0436</max_angle> <!-- 2.5 degree -->
-	          </horizontal>
-<!--            Can't use vertical rays until this bug is resolved: -->
-<!--            https://bitbucket.org/osrf/gazebo/issue/509/vertical-sensor-doesnt-works -->
-<!-- 	          <vertical> -->
-<!-- 	            <samples>50</samples> -->
-<!-- 	            <resolution>1.0</resolution> -->
-<!-- 	            <min_angle>-0.0436</min_angle>  -2.5 degree -->
-<!-- 	            <max_angle>0.0436</max_angle> 2.5 degree -->
-<!-- 	          </vertical> -->
-	        </scan>
-	        <range>
-	          <min>0.01</min>
-	          <max>0.15</max>
-	          <resolution>1.0</resolution>
-	        </range>
-	      </ray>
-	    </sensor>
-	  </gazebo>
-	  <gazebo reference="cliff_sensor_right_link">
-	    <sensor type="ray" name="cliff_sensor_right">
-	      <always_on>true</always_on>
-	      <update_rate>50</update_rate>
-	      <visualize>true</visualize>
-	      <ray>
-	        <scan>
-	          <horizontal>
-	            <samples>50</samples>
-	            <resolution>1.0</resolution>
-	            <min_angle>-0.0436</min_angle>  <!-- -2.5 degree -->
-	            <max_angle>0.0436</max_angle> <!-- 2.5 degree -->
-	          </horizontal>
-<!--            Can't use vertical rays until this bug is resolved: -->
-<!--            https://bitbucket.org/osrf/gazebo/issue/509/vertical-sensor-doesnt-works -->
-<!-- 	          <vertical> -->
-<!-- 	            <samples>50</samples> -->
-<!-- 	            <resolution>1.0</resolution> -->
-<!-- 	            <min_angle>-0.0436</min_angle>  -2.5 degree -->
-<!-- 	            <max_angle>0.0436</max_angle> 2.5 degree -->
-<!-- 	          </vertical> -->
-	        </scan>
-	        <range>
-	          <min>0.01</min>
-	          <max>0.15</max>
-	          <resolution>1.0</resolution>
-	        </range>
-	      </ray>
-	    </sensor>
-	  </gazebo>
-	  <gazebo reference="cliff_sensor_front_link">
-	    <sensor type="ray" name="cliff_sensor_front">
-	      <always_on>true</always_on>
-	      <update_rate>50</update_rate>
-	      <visualize>true</visualize>
-	      <ray>
-	        <scan>
-	          <horizontal>
-	            <samples>50</samples>
-	            <resolution>1.0</resolution>
-	            <min_angle>-0.0436</min_angle>  <!-- -2.5 degree -->
-	            <max_angle>0.0436</max_angle> <!-- 2.5 degree -->
-	          </horizontal>
-<!-- 	          Can't use vertical rays until this bug is resolved: -->
-<!--            https://bitbucket.org/osrf/gazebo/issue/509/vertical-sensor-doesnt-works -->
-<!-- 	          <vertical> -->
-<!-- 	            <samples>50</samples> -->
-<!-- 	            <resolution>1.0</resolution> -->
-<!-- 	            <min_angle>-0.0436</min_angle>  -2.5 degree -->
-<!-- 	            <max_angle>0.0436</max_angle> 2.5 degree -->
-<!-- 	          </vertical> -->
-	        </scan>
-	        <range>
-	          <min>0.01</min>
-	          <max>0.15</max>
-	          <resolution>1.0</resolution>
-	        </range>
-	      </ray>
-	    </sensor>
-	  </gazebo>
-	  <gazebo reference="gyro_link">
-	   <sensor type="imu" name="imu">
-        <always_on>true</always_on>
-        <update_rate>50</update_rate>
-        <visualize>false</visualize>
-        <imu>
-          <noise>
-            <type>gaussian</type>
-	          <rate>
-	            <mean>0.0</mean>
-	            <stddev>${0.0014*0.0014}</stddev> <!-- 0.25 x 0.25 (deg/s) -->
-	            <bias_mean>0.0</bias_mean>
-	            <bias_stddev>0.0</bias_stddev>
-	          </rate>
-		        <accel> <!-- not used in the plugin and real robot, hence using tutorial values -->
-			        <mean>0.0</mean>
-			        <stddev>1.7e-2</stddev>
-			        <bias_mean>0.1</bias_mean>
-			        <bias_stddev>0.001</bias_stddev>
-		        </accel>
-          </noise>
-	      </imu>
-      </sensor>
-	  </gazebo>
-	  <gazebo>
-	    <plugin name="kobuki_controller" filename="libgazebo_ros_kobuki.so">
-	      <publish_tf>1</publish_tf>
-	      <left_wheel_joint_name>wheel_left_joint</left_wheel_joint_name>
-	      <right_wheel_joint_name>wheel_right_joint</right_wheel_joint_name>
-	      <wheel_separation>.230</wheel_separation>
-	      <wheel_diameter>0.070</wheel_diameter>
-	      <torque>1.0</torque>
-	      <velocity_command_timeout>0.6</velocity_command_timeout>
-	      <cliff_sensor_left_name>cliff_sensor_left</cliff_sensor_left_name>
-	      <cliff_sensor_center_name>cliff_sensor_front</cliff_sensor_center_name>
-	      <cliff_sensor_right_name>cliff_sensor_right</cliff_sensor_right_name>
-	      <cliff_detection_threshold>0.04</cliff_detection_threshold>
-	      <bumper_name>bumpers</bumper_name>
-        <imu_name>imu</imu_name>
-	    </plugin>
-	  </gazebo>
-  </xacro:macro>
+	<xacro:property name="deg_to_rad" value="0.01745329251994329577"/>
+	<xacro:property name="camera_name" value="camera"/>
+	<xacro:property name="topics_ns" value="camera"/>
+	<xacro:property name="color_optical_frame" value="${camera_name}_color_optical_frame"/>
+	<xacro:property name="depth_optical_frame" value="${camera_name}_depth_optical_frame"/>
+	<xacro:property name="infrared1_optical_frame" value="${camera_name}_left_ir_optical_frame"/>
+	<xacro:property name="infrared2_optical_frame" value="${camera_name}_right_ir_optical_frame"/>
+	<xacro:macro name="kobuki_sim">
+		<gazebo reference="wheel_left_link">
+			<mu1>1.0</mu1>
+			<mu2>1.0</mu2>
+			<kp>1000000.0</kp>
+			<kd>100.0</kd>
+			<minDepth>0.001</minDepth>
+			<maxVel>1.0</maxVel>
+		</gazebo>
+		<gazebo reference="wheel_right_link">
+			<mu1>1.0</mu1>
+			<mu2>1.0</mu2>
+			<kp>1000000.0</kp>
+			<kd>100.0</kd>
+			<minDepth>0.001</minDepth>
+			<maxVel>1.0</maxVel>
+		</gazebo>
+		<gazebo reference="caster_front_link">
+			<mu1>0.0</mu1>
+			<mu2>0.0</mu2>
+			<kp>1000000.0</kp>
+			<kd>100.0</kd>
+			<minDepth>0.001</minDepth>
+			<maxVel>1.0</maxVel>
+		</gazebo>
+		<gazebo reference="caster_back_link">
+			<mu1>0.0</mu1>
+			<mu2>0.0</mu2>
+			<kp>1000000.0</kp>
+			<kd>100.0</kd>
+			<minDepth>0.001</minDepth>
+			<maxVel>1.0</maxVel>
+		</gazebo>
+		<gazebo reference="base_link">
+			<mu1>0.3</mu1>
+			<mu2>0.3</mu2>
+			<sensor type="contact" name="bumpers">
+			<always_on>1</always_on>
+			<update_rate>50.0</update_rate>
+			<visualize>true</visualize>
+			<contact>
+				<collision>base_footprint_fixed_joint_lump__base_collision</collision>
+			</contact>
+			</sensor>
+		</gazebo>
+		<!-- depth camera-->
+		<gazebo reference="camera_link">
+			<self_collide>0</self_collide>
+			<enable_wind>0</enable_wind>
+			<kinematic>0</kinematic>
+			<gravity>1</gravity>
+			<!--<mu>1</mu>-->
+			<mu2>1</mu2>
+			<fdir1>0 0 0</fdir1>
+			<!--<slip1>0</slip1>
+			<slip2>0</slip2>-->
+			<kp>1e+13</kp>
+			<kd>1</kd>
+			<!--<max_vel>0.01</max_vel>
+			<min_depth>0</min_depth>-->
+			<sensor name="${camera_name}color" type="camera">
+			<camera name="${camera_name}">
+				<horizontal_fov>${69.4*deg_to_rad}</horizontal_fov>
+				<image>
+				<width>1920</width>
+				<height>1080</height>
+				<format>RGB_INT8</format>
+				</image>
+				<clip>
+				<near>0.1</near>
+				<far>100</far>
+				</clip>
+				<noise>
+				<type>gaussian</type>
+				<mean>0.0</mean>
+				<stddev>0.007</stddev>
+				</noise>
+			</camera>
+			<always_on>1</always_on>
+			<update_rate>30</update_rate>
+			<visualize>1</visualize>
+			</sensor>
+			<sensor name="${camera_name}ired1" type="camera">
+			<camera name="${camera_name}">
+				<horizontal_fov>${85.2*deg_to_rad}</horizontal_fov>
+				<image>
+				<width>1280</width>
+				<height>720</height>
+				<format>L_INT8</format>
+				</image>
+				<clip>
+				<near>0.1</near>
+				<far>100</far>
+				</clip>
+				<noise>
+				<type>gaussian</type>
+				<mean>0.0</mean>
+				<stddev>0.05</stddev>
+				</noise>
+			</camera>
+			<always_on>1</always_on>
+			<update_rate>90</update_rate>
+			<visualize>0</visualize>
+			</sensor>
+			<sensor name="${camera_name}ired2" type="camera">
+			<camera name="${camera_name}">
+				<horizontal_fov>${85.2*deg_to_rad}</horizontal_fov>
+				<image>
+				<width>1280</width>
+				<height>720</height>
+				<format>L_INT8</format>
+				</image>
+				<clip>
+				<near>0.1</near>
+				<far>100</far>
+				</clip>
+				<noise>
+				<type>gaussian</type>
+				<mean>0.0</mean>
+				<stddev>0.05</stddev>
+				</noise>
+			</camera>
+			<always_on>1</always_on>
+			<update_rate>90</update_rate>
+			<visualize>0</visualize>
+			</sensor>
+			<sensor name="${camera_name}depth" type="depth">
+			<camera name="${camera_name}">
+				<horizontal_fov>${85.2*deg_to_rad}</horizontal_fov>
+				<image>
+				<width>1280</width>
+				<height>720</height>
+				</image>
+				<clip>
+				<near>0.1</near>
+				<far>100</far>
+				</clip>
+				<noise>
+				<type>gaussian</type>
+				<mean>0.0</mean>
+				<stddev>0.100</stddev>
+				</noise>
+			</camera>
+			<always_on>1</always_on>
+			<update_rate>90</update_rate>
+			<visualize>0</visualize>
+			</sensor>
+		</gazebo>
+		<gazebo>
+			<plugin name="${topics_ns}" filename="librealsense_gazebo_plugin.so">
+				<prefix>${camera_name}</prefix>
+				<depthUpdateRate>60.0</depthUpdateRate>
+				<colorUpdateRate>60.0</colorUpdateRate>
+				<infraredUpdateRate>60.0</infraredUpdateRate>
+				<depthTopicName>depth/image_raw</depthTopicName>
+				<depthCameraInfoTopicName>depth/camera_info</depthCameraInfoTopicName>
+				<colorTopicName>color/image_raw</colorTopicName>
+				<colorCameraInfoTopicName>color/camera_info</colorCameraInfoTopicName>
+				<infrared1TopicName>infra1/image_raw</infrared1TopicName>
+				<infrared1CameraInfoTopicName>infra1/camera_info</infrared1CameraInfoTopicName>
+				<infrared2TopicName>infra2/image_raw</infrared2TopicName>
+				<infrared2CameraInfoTopicName>infra2/camera_info</infrared2CameraInfoTopicName>
+				<colorOpticalframeName>${color_optical_frame}</colorOpticalframeName>
+				<depthOpticalframeName>${depth_optical_frame}</depthOpticalframeName>
+				<infrared1OpticalframeName>${infrared1_optical_frame}</infrared1OpticalframeName>
+				<infrared2OpticalframeName>${infrared2_optical_frame}</infrared2OpticalframeName>
+				<rangeMinDepth>0.2</rangeMinDepth>
+				<rangeMaxDepth>10.0</rangeMaxDepth>
+				<pointCloud>true</pointCloud>
+				<pointCloudTopicName>depth/points</pointCloudTopicName>
+				<pointCloudCutoff>0.5</pointCloudCutoff>
+			</plugin>
+		</gazebo>
+		<!-- hokuyo -->
+		<gazebo reference="laser">
+		<sensor type="ray" name="head_hokuyo_sensor">
+			<pose>0 0 0.064 0 0 0</pose>
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
Commit message: laser merged functional

File: jaime_description/urdf/jaime.urdf.xacro (robot description, xacro)
@@ -244,5 +244,5 @@
     <!-- camera body, with origin at bottom screw mount -->
     <joint name="camera_joint" type="fixed">
-      <origin xyz="0.0 0.0 0.85" rpy="0 0.610865 0"/>
+      <origin xyz="0.0 0.0 1.0" rpy="0 0.610865 0"/>
       <parent link="base_link"/>
       <child link="camera_bottom_screw_frame" />

File: jaime_description/urdf/jaime_gazebo.urdf.xacro (robot description, xacro)
@@ -212,5 +212,5 @@
 			</ray>
 			<plugin name="gazebo_ros_head_hokuyo_controller" filename="libgazebo_ros_laser.so">
-			<topicName>scan</topicName>
+			<topicName>scan/hokuyo</topicName>
 			<frameName>laser</frameName>
 			</plugin>

Commit message: update urdf

File: jaime_description/urdf/jaime.urdf.xacro (robot description, xacro)
@@ -244,5 +244,5 @@
     <!-- camera body, with origin at bottom screw mount -->
     <joint name="camera_joint" type="fixed">
-      <origin xyz="0.0 0.0 1.0" rpy="0 0.610865 0"/>
+      <origin xyz="0.07 0.045 0.68" rpy="0 0 0"/>
       <parent link="base_link"/>
       <child link="camera_bottom_screw_frame" />

File: jaime_description/urdf/jaime_gazebo.urdf.xacro (robot description, xacro)
@@ -185,5 +185,5 @@
 		<sensor type="ray" name="head_hokuyo_sensor">
 			<pose>0 0 0.064 0 0 0</pose>
-			<visualize>true</visualize>
+			<visualize>false</visualize>
 			<update_rate>40</update_rate>
 			<ray>
