Commit message: (MA) solucionando CMake

File: jaime_description/urdf/jaime.xacro (robot description, xacro)
@@ -1,4 +1,4 @@
 <?xml version="1.0" ?>
-<robot name="bender" xmlns:xacro="http://www.ros.org/wiki/xacro">
+<robot name="jaime" xmlns:xacro="http://www.ros.org/wiki/xacro">
 <link name="base_link">
   <!--
@@ -12,5 +12,5 @@
     <origin xyz="0 0 0" rpy="0 0 0"/>
     <geometry>
-      <mesh filename="package://bender_description/meshes/base_link.stl" scale="0.001 0.001 0.001"/>
+      <mesh filename="package://jaime_description/meshes/base_link.stl" scale="0.001 0.001 0.001"/>
     </geometry>
     <material name="chassis_material">
@@ -21,5 +21,5 @@
     <origin xyz="0 0 0" rpy="0 0 0"/>
     <geometry>
-      <mesh filename="package://bender_description/meshes/base_link.stl" scale="0.001 0.001 0.001"/>
+      <mesh filename="package://jaime_description/meshes/base_link.stl" scale="0.001 0.001 0.001"/>
     </geometry>
   </collision>
@@ -40,5 +40,5 @@
     <origin xyz="-0.035737 -0.247634 -1.04582" rpy="0 0 0"/>
     <geometry>
-      <mesh filename="package://bender_description/meshes/l2l_1.stl" scale="0.001 0.001 0.001"/>
+      <mesh filename="package://jaime_description/meshes/l2l_1.stl" scale="0.001 0.001 0.001"/>
     </geometry>
     <material name="chassis_material">
@@ -49,5 +49,5 @@
     <origin xyz="-0.035737 -0.247634 -1.04582" rpy="0 0 0"/>
     <geometry>
-      <mesh filename="package://bender_description/meshes/l2l_1.stl" scale="0.001 0.001 0.001"/>
+      <mesh filename="package://jaime_description/meshes/l2l_1.stl" scale="0.001 0.001 0.001"/>
     </geometry>
   </collision>
@@ -62,5 +62,5 @@
     <origin xyz="-0.007987 -0.247634 -0.985406" rpy="0 0 0"/>
     <geometry>
-      <mesh filename="package://bender_description/meshes/l3l_1.stl" scale="0.001 0.001 0.001"/>
+      <mesh filename="package://jaime_description/meshes/l3l_1.stl" scale="0.001 0.001 0.001"/>
     </geometry>
     <material name="chassis_material">
@@ -71,5 +71,5 @@
     <origin xyz="-0.007987 -0.247634 -0.985406" rpy="0 0 0"/>
     <geometry>
-      <mesh filename="package://bender_description/meshes/l3l_1.stl" scale="0.001 0.001 0.001"/>
+      <mesh filename="package://jaime_description/meshes/l3l_1.stl" scale="0.001 0.001 0.001"/>
     </geometry>
   </collision>
@@ -84,5 +84,5 @@
     <origin xyz="-0.006819 -0.275388 -0.815556" rpy="0 0 0"/>
     <geometry>
-      <mesh filename="package://bender_description/meshes/l4l_1.stl" scale="0.001 0.001 0.001"/>
+      <mesh filename="package://jaime_description/meshes/l4l_1.stl" scale="0.001 0.001 0.001"/>
     </geometry>
     <material name="chassis_material">
@@ -93,5 +93,5 @@
     <origin xyz="-0.006819 -0.275388 -0.815556" rpy="0 0 0"/>
     <geometry>
-      <mesh filename="package://bender_description/meshes/l4l_1.stl" scale="0.001 0.001 0.001"/>
+      <mesh filename="package://jaime_description/meshes/l4l_1.stl" scale="0.001 0.001 0.001"/>
     </geometry>
   </collision>
@@ -106,5 +106,5 @@
     <origin xyz="-0.006819 -0.247637 -0.767806" rpy="0 0 0"/>
     <geometry>
-      <mesh filename="package://bender_description/meshes/l5l_1.stl" scale="0.001 0.001 0.001"/>
+      <mesh filename="package://jaime_description/meshes/l5l_1.stl" scale="0.001 0.001 0.001"/>
     </geometry>
     <material name="chassis_material">
@@ -115,5 +115,5 @@
     <origin xyz="-0.006819 -0.247637 -0.767806" rpy="0 0 0"/>
     <geometry>
-      <mesh filename="package://bender_description/meshes/l5l_1.stl" scale="0.001 0.001 0.001"/>
+      <mesh filename="package://jaime_description/meshes/l5l_1.stl" scale="0.001 0.001 0.001"/>
     </geometry>
   </collision>
@@ -128,5 +128,5 @@
     <origin xyz="-0.007275 -0.269887 -0.504262" rpy="0 0 0"/>
     <geometry>
-      <mesh filename="package://bender_description/meshes/l6l_1.stl" scale="0.001 0.001 0.001"/>
+      <mesh filename="package://jaime_description/meshes/l6l_1.stl" scale="0.001 0.001 0.001"/>
     </geometry>
     <material name="chassis_material">
@@ -137,5 +137,5 @@
     <origin xyz="-0.007275 -0.269887 -0.504262" rpy="0 0 0"/>
     <geometry>
-      <mesh filename="package://bender_description/meshes/l6l_1.stl" scale="0.001 0.001 0.001"/>
+      <mesh filename="package://jaime_description/meshes/l6l_1.stl" scale="0.001 0.001 0.001"/>
     </geometry>
   </collision>
@@ -150,5 +150,5 @@
     <origin xyz="-0.035737 0.262366 -1.04582" rpy="0 0 0"/>
     <geometry>
-      <mesh filename="package://bender_description/meshes/l2r_1.stl" scale="0.001 0.001 0.001"/>
+      <mesh filename="package://jaime_description/meshes/l2r_1.stl" scale="0.001 0.001 0.001"/>
     </geometry>
     <material name="chassis_material">
@@ -159,5 +159,5 @@
     <origin xyz="-0.035737 0.262366 -1.04582" rpy="0 0 0"/>
     <geometry>
-      <mesh filename="package://bender_description/meshes/l2r_1.stl" scale="0.001 0.001 0.001"/>
+      <mesh filename="package://jaime_description/meshes/l2r_1.stl" scale="0.001 0.001 0.001"/>
     </geometry>
   </collision>
@@ -172,5 +172,5 @@
     <origin xyz="-0.007987 0.262366 -0.985406" rpy="0 0 0"/>
     <geometry>
-      <mesh filename="package://bender_description/meshes/l3r_1.stl" scale="0.001 0.001 0.001"/>
+      <mesh filename="package://jaime_description/meshes/l3r_1.stl" scale="0.001 0.001 0.001"/>
     </geometry>
     <material name="chassis_material">
@@ -181,5 +181,5 @@
     <origin xyz="-0.007987 0.262366 -0.985406" rpy="0 0 0"/>
     <geometry>
-      <mesh filename="package://bender_description/meshes/l3r_1.stl" scale="0.001 0.001 0.001"/>
+      <mesh filename="package://jaime_description/meshes/l3r_1.stl" scale="0.001 0.001 0.001"/>
     </geometry>
   </collision>
@@ -194,5 +194,5 @@
     <origin xyz="-0.006819 0.290116 -0.815556" rpy="0 0 0"/>
     <geometry>
-      <mesh filename="package://bender_description/meshes/l4r_1.stl" scale="0.001 0.001 0.001"/>
+      <mesh filename="package://jaime_description/meshes/l4r_1.stl" scale="0.001 0.001 0.001"/>
     </geometry>
     <material name="chassis_material">
@@ -203,5 +203,5 @@
     <origin xyz="-0.006819 0.290116 -0.815556" rpy="0 0 0"/>
     <geometry>
-      <mesh filename="package://bender_description/meshes/l4r_1.stl" scale="0.001 0.001 0.001"/>
+      <mesh filename="package://jaime_description/meshes/l4r_1.stl" scale="0.001 0.001 0.001"/>
     </geometry>
   </collision>
@@ -216,5 +216,5 @@
     <origin xyz="-0.006819 0.262364 -0.767806" rpy="0 0 0"/>
     <geometry>
-      <mesh filename="package://bender_description/meshes/l5r_1.stl" scale="0.001 0.001 0.001"/>
+      <mesh filename="package://jaime_description/meshes/l5r_1.stl" scale="0.001 0.001 0.001"/>
     </geometry>
     <material name="chassis_material">
@@ -225,5 +225,5 @@
     <origin xyz="-0.006819 0.262364 -0.767806" rpy="0 0 0"/>
     <geometry>
-      <mesh filename="package://bender_description/meshes/l5r_1.stl" scale="0.001 0.001 0.001"/>
+      <mesh filename="package://jaime_description/meshes/l5r_1.stl" scale="0.001 0.001 0.001"/>
     </geometry>
   </collision>
@@ -238,5 +238,5 @@
     <origin xyz="-0.007275 0.284614 -0.504262" rpy="0 0 0"/>
     <geometry>
-      <mesh filename="package://bender_description/meshes/l6r_1.stl" scale="0.001 0.001 0.001"/>
+      <mesh filename="package://jaime_description/meshes/l6r_1.stl" scale="0.001 0.001 0.001"/>
     </geometry>
     <material name="chassis_material">
@@ -247,5 +247,5 @@
     <origin xyz="-0.007275 0.284614 -0.504262" rpy="0 0 0"/>
     <geometry>
-      <mesh filename="package://bender_description/meshes/l6r_1.stl" scale="0.001 0.001 0.001"/>
+      <mesh filename="package://jaime_description/meshes/l6r_1.stl" scale="0.001 0.001 0.001"/>
     </geometry>
   </collision>
@@ -260,5 +260,5 @@
     <origin xyz="-0.007987 0.037366 -1.28382" rpy="0 0 0"/>
     <geometry>
-      <mesh filename="package://bender_description/meshes/l2h_1.stl" scale="0.001 0.001 0.001"/>
+      <mesh filename="package://jaime_description/meshes/l2h_1.stl" scale="0.001 0.001 0.001"/>
     </geometry>
     <material name="chassis_material">
@@ -269,5 +269,5 @@
     <origin xyz="-0.007987 0.037366 -1.28382" rpy="0 0 0"/>
     <geometry>
-      <mesh filename="package://bender_description/meshes/l2h_1.stl" scale="0.001 0.001 0.001"/>
+      <mesh filename="package://jaime_description/meshes/l2h_1.stl" scale="0.001 0.001 0.001"/>
     </geometry>
   </collision>
@@ -282,5 +282,5 @@
     <origin xyz="-0.049487 0.007366 -1.40882" rpy="0 0 0"/>
     <geometry>
-      <mesh filename="package://bender_description/meshes/real_sense_1.stl" scale="0.001 0.001 0.001"/>
+      <mesh filename="package://jaime_description/meshes/real_sense_1.stl" scale="0.001 0.001 0.001"/>
     </geometry>
     <material name="chassis_material">
@@ -291,5 +291,5 @@
     <origin xyz="-0.049487 0.007366 -1.40882" rpy="0 0 0"/>
     <geometry>
-      <mesh filename="package://bender_description/meshes/real_sense_1.stl" scale="0.001 0.001 0.001"/>
+      <mesh filename="package://jaime_description/meshes/real_sense_1.stl" scale="0.001 0.001 0.001"/>
     </geometry>
   </collision>
@@ -304,5 +304,5 @@
     <origin xyz="-0.007275 0.262364 -0.480247" rpy="0 0 0"/>
     <geometry>
-      <mesh filename="package://bender_description/meshes/g1r_1.stl" scale="0.001 0.001 0.001"/>
+      <mesh filename="package://jaime_description/meshes/g1r_1.stl" scale="0.001 0.001 0.001"/>
     </geometry>
     <material name="chassis_material">
@@ -313,5 +313,5 @@
     <origin xyz="-0.007275 0.262364 -0.480247" rpy="0 0 0"/>
     <geometry>
-      <mesh filename="package://bender_description/meshes/g1r_1.stl" scale="0.001 0.001 0.001"/>
+      <mesh filename="package://jaime_description/meshes/g1r_1.stl" scale="0.001 0.001 0.001"/>
     </geometry>
   </collision>
@@ -326,5 +326,5 @@
     <origin xyz="-0.029225 0.243864 -0.438647" rpy="0 0 0"/>
     <geometry>
-      <mesh filename="package://bender_description/meshes/g2ra_1.stl" scale="0.001 0.001 0.001"/>
+      <mesh filename="package://jaime_description/meshes/g2ra_1.stl" scale="0.001 0.001 0.001"/>
     </geometry>
     <material name="chassis_material">
@@ -335,5 +335,5 @@
     <origin xyz="-0.029225 0.243864 -0.438647" rpy="0 0 0"/>
     <geometry>
-      <mesh filename="package://bender_description/meshes/g2ra_1.stl" scale="0.001 0.001 0.001"/>
+      <mesh filename="package://jaime_description/meshes/g2ra_1.stl" scale="0.001 0.001 0.001"/>
     </geometry>
   </collision>
@@ -348,5 +348,5 @@
     <origin xyz="-0.029225 0.280864 -0.438647" rpy="0 0 0"/>
     <geometry>
-      <mesh filename="package://bender_description/meshes/g2rb_1.stl" scale="0.001 0.001 0.001"/>
+      <mesh filename="package://jaime_description/meshes/g2rb_1.stl" scale="0.001 0.001 0.001"/>
     </geometry>
     <material name="chassis_material">
@@ -357,5 +357,5 @@
     <origin xyz="-0.029225 0.280864 -0.438647" rpy="0 0 0"/>
     <geometry>
-      <mesh filename="package://bender_description/meshes/g2rb_1.stl" scale="0.001 0.001 0.001"/>
+      <mesh filename="package://jaime_description/meshes/g2rb_1.stl" scale="0.001 0.001 0.001"/>
     </geometry>
   </collision>
@@ -370,5 +370,5 @@
     <origin xyz="-0.007275 -0.247637 -0.480247" rpy="0 0 0"/>
     <geometry>
-      <mesh filename="package://bender_description/meshes/g1l_1.stl" scale="0.001 0.001 0.001"/>
+      <mesh filename="package://jaime_description/meshes/g1l_1.stl" scale="0.001 0.001 0.001"/>
     </geometry>
     <material name="chassis_material">
@@ -379,5 +379,5 @@
     <origin xyz="-0.007275 -0.247637 -0.480247" rpy="0 0 0"/>
     <geometry>
-      <mesh filename="package://bender_description/meshes/g1l_1.stl" scale="0.001 0.001 0.001"/>
+      <mesh filename="package://jaime_description/meshes/g1l_1.stl" scale="0.001 0.001 0.001"/>
     </geometry>
   </collision>
@@ -392,5 +392,5 @@
     <origin xyz="-0.029225 -0.266137 -0.438647" rpy="0 0 0"/>
     <geometry>
-      <mesh filename="package://bender_description/meshes/g2lb_1.stl" scale="0.001 0.001 0.001"/>
+      <mesh filename="package://jaime_description/meshes/g2lb_1.stl" scale="0.001 0.001 0.001"/>
     </geometry>
     <material name="chassis_material">
@@ -401,5 +401,5 @@
     <origin xyz="-0.029225 -0.266137 -0.438647" rpy="0 0 0"/>
     <geometry>
-      <mesh filename="package://bender_description/meshes/g2lb_1.stl" scale="0.001 0.001 0.001"/>
+      <mesh filename="package://jaime_description/meshes/g2lb_1.stl" scale="0.001 0.001 0.001"/>
     </geometry>
   </collision>
@@ -414,5 +414,5 @@
     <origin xyz="-0.029225 -0.229137 -0.438647" rpy="0 0 0"/>
     <geometry>
-      <mesh filename="package://bender_description/meshes/g2la_1.stl" scale="0.001 0.001 0.001"/>
+      <mesh filename="package://jaime_description/meshes/g2la_1.stl" scale="0.001 0.001 0.001"/>
     </geometry>
     <material name="chassis_material">
@@ -423,5 +423,5 @@
     <origin xyz="-0.029225 -0.229137 -0.438647" rpy="0 0 0"/>
     <geometry>
-      <mesh filename="package://bender_description/meshes/g2la_1.stl" scale="0.001 0.001 0.001"/>
+      <mesh filename="package://jaime_description/meshes/g2la_1.stl" scale="0.001 0.001 0.001"/>
     </geometry>
   </collision>
@@ -436,5 +436,5 @@
     <origin xyz="-0.188322 0.007366 -0.25882" rpy="0 0 0"/>
     <geometry>
-      <mesh filename="package://bender_description/meshes/laser_1.stl" scale="0.001 0.001 0.001"/>
+      <mesh filename="package://jaime_description/meshes/laser_1.stl" scale="0.001 0.001 0.001"/>
     </geometry>
     <material name="chassis_material">
@@ -445,5 +445,5 @@
     <origin xyz="-0.188322 0.007366 -0.25882" rpy="0 0 0"/>
     <geometry>
-      <mesh filename="package://bender_description/meshes/laser_1.stl" scale="0.001 0.001 0.001"/>
+      <mesh filename="package://jaime_description/meshes/laser_1.stl" scale="0.001 0.001 0.001"/>
     </geometry>
   </collision>
@@ -458,5 +458,5 @@
     <origin xyz="-0.135487 0.164865 -0.09982" rpy="0 0 0"/>
     <geometry>
-      <mesh filename="package://bender_description/meshes/wfr_1.stl" scale="0.001 0.001 0.001"/>
+      <mesh filename="package://jaime_description/meshes/wfr_1.stl" scale="0.001 0.001 0.001"/>
     </geometry>
     <material name="chassis_material">
@@ -467,5 +467,5 @@
     <origin xyz="-0.135487 0.164865 -0.09982" rpy="0 0 0"/>
     <geometry>
-      <mesh filename="package://bender_description/meshes/wfr_1.stl" scale="0.001 0.001 0.001"/>
+      <mesh filename="package://jaime_description/meshes/wfr_1.stl" scale="0.001 0.001 0.001"/>
     </geometry>
   </collision>
@@ -480,5 +480,5 @@
     <origin xyz="0.114513 0.164865 -0.09982" rpy="0 0 0"/>
     <geometry>
-      <mesh filename="package://bender_description/meshes/wrr_1.stl" scale="0.001 0.001 0.001"/>
+      <mesh filename="package://jaime_description/meshes/wrr_1.stl" scale="0.001 0.001 0.001"/>
     </geometry>
     <material name="chassis_material">
@@ -489,5 +489,5 @@
     <origin xyz="0.114513 0.164865 -0.09982" rpy="0 0 0"/>
     <geometry>
-      <mesh filename="package://bender_description/meshes/wrr_1.stl" scale="0.001 0.001 0.001"/>
+      <mesh filename="package://jaime_description/meshes/wrr_1.stl" scale="0.001 0.001 0.001"/>
     </geometry>
   </collision>
@@ -502,5 +502,5 @@
     <origin xyz="-0.135487 -0.150135 -0.09982" rpy="0 0 0"/>
     <geometry>
-      <mesh filename="package://bender_description/meshes/wfl_1.stl" scale="0.001 0.001 0.001"/>
+      <mesh filename="package://jaime_description/meshes/wfl_1.stl" scale="0.001 0.001 0.001"/>
     </geometry>
     <material name="chassis_material">
@@ -511,5 +511,5 @@
     <origin xyz="-0.135487 -0.150135 -0.09982" rpy="0 0 0"/>
     <geometry>
-      <mesh filename="package://bender_description/meshes/wfl_1.stl" scale="0.001 0.001 0.001"/>
+      <mesh filename="package://jaime_description/meshes/wfl_1.stl" scale="0.001 0.001 0.001"/>
     </geometry>
   </collision>
@@ -524,5 +524,5 @@
     <origin xyz="0.114513 -0.150135 -0.09982" rpy="0 0 0"/>
     <geometry>
-      <mesh filename="package://bender_description/meshes/wrl_1.stl" scale="0.001 0.001 0.001"/>
+      <mesh filename="package://jaime_description/meshes/wrl_1.stl" scale="0.001 0.001 0.001"/>
     </geometry>
     <material name="chassis_material">
@@ -533,5 +533,5 @@
     <origin xyz="0.114513 -0.150135 -0.09982" rpy="0 0 0"/>
     <geometry>
-      <mesh filename="package://bender_description/meshes/wrl_1.stl" scale="0.001 0.001 0.001"/>
+      <mesh filename="package://jaime_description/meshes/wrl_1.stl" scale="0.001 0.001 0.001"/>
     </geometry>
   </collision>
@@ -546,5 +546,5 @@
     <origin xyz="-0.007987 0.227866 -1.06382" rpy="0 0 0"/>
     <geometry>
-      <mesh filename="package://bender_description/meshes/l1r_1.stl" scale="0.001 0.001 0.001"/>
+      <mesh filename="package://jaime_description/meshes/l1r_1.stl" scale="0.001 0.001 0.001"/>
     </geometry>
     <material name="chassis_material">
@@ -555,5 +555,5 @@
     <origin xyz="-0.007987 0.227866 -1.06382" rpy="0 0 0"/>
     <geometry>
-      <mesh filename="package://bender_description/meshes/l1r_1.stl" scale="0.001 0.001 0.001"/>
+      <mesh filename="package://jaime_description/meshes/l1r_1.stl" scale="0.001 0.001 0.001"/>
     </geometry>
   </collision>
@@ -568,5 +568,5 @@
     <origin xyz="-0.007987 -0.213134 -1.06382" rpy="0 0 0"/>
     <geometry>
-      <mesh filename="package://bender_description/meshes/l1l_1.stl" scale="0.001 0.001 0.001"/>
+      <mesh filename="package://jaime_description/meshes/l1l_1.stl" scale="0.001 0.001 0.001"/>
     </geometry>
     <material name="chassis_material">
@@ -577,5 +577,5 @@
     <origin xyz="-0.007987 -0.213134 -1.06382" rpy="0 0 0"/>
     <geometry>
-      <mesh filename="package://bender_description/meshes/l1l_1.stl" scale="0.001 0.001 0.001"/>
+      <mesh filename="package://jaime_description/meshes/l1l_1.stl" scale="0.001 0.001 0.001"/>
     </geometry>
   </collision>
@@ -590,5 +590,5 @@
     <origin xyz="-0.007987 0.007366 -1.21382" rpy="0 0 0"/>
     <geometry>
-      <mesh filename="package://bender_description/meshes/l1h_1.stl" scale="0.001 0.001 0.001"/>
+      <mesh filename="package://jaime_description/meshes/l1h_1.stl" scale="0.001 0.001 0.001"/>
     </geometry>
     <material name="chassis_material">
@@ -599,5 +599,5 @@
     <origin xyz="-0.007987 0.007366 -1.21382" rpy="0 0 0"/>
     <geometry>
-      <mesh filename="package://bender_description/meshes/l1h_1.stl" scale="0.001 0.001 0.001"/>
+      <mesh filename="package://jaime_description/meshes/l1h_1.stl" scale="0.001 0.001 0.001"/>
     </geometry>
   </collision>

File: jaime_description/urdf/materials.xacro (robot description, xacro)
@@ -1,4 +1,4 @@
 <?xml version="1.0" ?>
-<robot name="bender" xmlns:xacro="http://www.ros.org/wiki/xacro" >
+<robot name="jaime" xmlns:xacro="http://www.ros.org/wiki/xacro" >
 <material name="silver">
   <color rgba="0.700 0.700 0.700 1.000"/>
