Commit message: (MA) preparando jaime para navegacion

File: jaime_description/urdf/jaime.xacro (robot description, xacro)
@@ -31,782 +31,2 @@
   <origin xyz="0 0 0" rpy="0 0 0"/>
 </joint>
-<link name="l2l_1">
-  <inertial>
-    <origin xyz="-0.008469138038562633 4.816697341814002e-07 -0.07819087904751898" rpy="0 0 0"/>
-    <mass value="0.14071836856258027"/>
-    <inertia ixx="9.8e-05" iyy="0.000118" izz="8.7e-05" ixy="-0.0" iyz="-0.0" ixz="1.7e-05"/>
-  </inertial>
-  <visual>
-    <origin xyz="-0.035737 -0.247634 -1.04582" rpy="0 0 0"/>
-    <geometry>
-      <mesh filename="package://jaime_description/meshes/l2l_1.stl" scale="0.001 0.001 0.001"/>
-    </geometry>
-    <material name="chassis_material">
-      <color rgba="0.75 0.75 0.75 1.0"/>
-    </material>
-  </visual>
-  <collision>
-    <origin xyz="-0.035737 -0.247634 -1.04582" rpy="0 0 0"/>
-    <geometry>
-      <mesh filename="package://jaime_description/meshes/l2l_1.stl" scale="0.001 0.001 0.001"/>
-    </geometry>
-  </collision>
-</link>
-<link name="l3l_1">
-  <inertial>
-    <origin xyz="-0.004049240589701097 -0.00011662761889197348 -0.1333626785766504" rpy="0 0 0"/>
-    <mass value="0.13433192894969845"/>
-    <inertia ixx="0.000296" iyy="0.000299" izz="4.9e-05" ixy="0.0" iyz="-0.0" ixz="4e-05"/>
-  </inertial>
-  <visual>
-    <origin xyz="-0.007987 -0.247634 -0.985406" rpy="0 0 0"/>
-    <geometry>
-      <mesh filename="package://jaime_description/meshes/l3l_1.stl" scale="0.001 0.001 0.001"/>
-    </geometry>
-    <material name="chassis_material">
-      <color rgba="0.75 0.75 0.75 1.0"/>
-    </material>
-  </visual>
-  <collision>
-    <origin xyz="-0.007987 -0.247634 -0.985406" rpy="0 0 0"/>
-    <geometry>
-      <mesh filename="package://jaime_description/meshes/l3l_1.stl" scale="0.001 0.001 0.001"/>
-    </geometry>
-  </collision>
-</link>
-<link name="l4l_1">
-  <inertial>
-    <origin xyz="-0.022033052289373113 -0.027751420924878867 -0.07009451131427447" rpy="0 0 0"/>
-    <mass value="0.1319735958452518"/>
-    <inertia ixx="6.8e-05" iyy="8e-05" izz="7.4e-05" ixy="-0.0" iyz="0.0" ixz="-2e-06"/>
-  </inertial>
-  <visual>
-    <origin xyz="-0.006819 -0.275388 -0.815556" rpy="0 0 0"/>
-    <geometry>
-      <mesh filename="package://jaime_description/meshes/l4l_1.stl" scale="0.001 0.001 0.001"/>
-    </geometry>
-    <material name="chassis_material">
-      <color rgba="0.75 0.75 0.75 1.0"/>
-    </material>
-  </visual>
-  <collision>
-    <origin xyz="-0.006819 -0.275388 -0.815556" rpy="0 0 0"/>
-    <geometry>
-      <mesh filename="package://jaime_description/meshes/l4l_1.stl" scale="0.001 0.001 0.001"/>
-    </geometry>
-  </collision>
-</link>
-<link name="l5l_1">
-  <inertial>
-    <origin xyz="0.0039138191304953236 -6.519106588914747e-05 -0.1904912654580233" rpy="0 0 0"/>
-    <mass value="0.09538513786529154"/>
-    <inertia ixx="0.000748" iyy="0.000753" izz="3e-05" ixy="-0.0" iyz="-0.0" ixz="-5.3e-05"/>
-  </inertial>
-  <visual>
-    <origin xyz="-0.006819 -0.247637 -0.767806" rpy="0 0 0"/>
-    <geometry>
-      <mesh filename="package://jaime_description/meshes/l5l_1.stl" scale="0.001 0.001 0.001"/>
-    </geometry>
-    <material name="chassis_material">
-      <color rgba="0.75 0.75 0.75 1.0"/>
-    </material>
-  </visual>
-  <collision>
-    <origin xyz="-0.006819 -0.247637 -0.767806" rpy="0 0 0"/>
-    <geometry>
-      <mesh filename="package://jaime_description/meshes/l5l_1.stl" scale="0.001 0.001 0.001"/>
-    </geometry>
-  </collision>
-</link>
-<link name="l6l_1">
-  <inertial>
-    <origin xyz="1.1454305421428751e-07 -0.02225042100756011 -0.015076116417847174" rpy="0 0 0"/>
-    <mass value="0.004187419664904639"/>
-    <inertia ixx="2e-06" iyy="1e-06" izz="2e-06" ixy="-0.0" iyz="0.0" ixz="-0.0"/>
-  </inertial>
-  <visual>
-    <origin xyz="-0.007275 -0.269887 -0.504262" rpy="0 0 0"/>
-    <geometry>
-      <mesh filename="package://jaime_description/meshes/l6l_1.stl" scale="0.001 0.001 0.001"/>
-    </geometry>
-    <material name="chassis_material">
-      <color rgba="0.75 0.75 0.75 1.0"/>
-    </material>
-  </visual>
-  <collision>
-    <origin xyz="-0.007275 -0.269887 -0.504262" rpy="0 0 0"/>
-    <geometry>
-      <mesh filename="package://jaime_description/meshes/l6l_1.stl" scale="0.001 0.001 0.001"/>
-    </geometry>
-  </collision>
-</link>
-<link name="l2r_1">
-  <inertial>
-    <origin xyz="-0.008469138038563282 4.816697872778164e-07 -0.07819087904754218" rpy="0 0 0"/>
-    <mass value="0.14071836856258027"/>
-    <inertia ixx="9.8e-05" iyy="0.000118" izz="8.7e-05" ixy="-0.0" iyz="-0.0" ixz="1.7e-05"/>
-  </inertial>
-  <visual>
-    <origin xyz="-0.035737 0.262366 -1.04582" rpy="0 0 0"/>
-    <geometry>
-      <mesh filename="package://jaime_description/meshes/l2r_1.stl" scale="0.001 0.001 0.001"/>
-    </geometry>
-    <material name="chassis_material">
-      <color rgba="0.75 0.75 0.75 1.0"/>
-    </material>
-  </visual>
-  <collision>
-    <origin xyz="-0.035737 0.262366 -1.04582" rpy="0 0 0"/>
-    <geometry>
-      <mesh filename="package://jaime_description/meshes/l2r_1.stl" scale="0.001 0.001 0.001"/>
-    </geometry>
-  </collision>
-</link>
-<link name="l3r_1">
-  <inertial>
-    <origin xyz="-0.004049240589694631 -0.00011662761884700945 -0.1333626785766734" rpy="0 0 0"/>
-    <mass value="0.13433192894969845"/>
-    <inertia ixx="0.000296" iyy="0.000299" izz="4.9e-05" ixy="0.0" iyz="-0.0" ixz="4e-05"/>
-  </inertial>
-  <visual>
-    <origin xyz="-0.007987 0.262366 -0.985406" rpy="0 0 0"/>
-    <geometry>
-      <mesh filename="package://jaime_description/meshes/l3r_1.stl" scale="0.001 0.001 0.001"/>
-    </geometry>
-    <material name="chassis_material">
-      <color rgba="0.75 0.75 0.75 1.0"/>
-    </material>
-  </visual>
-  <collision>
-    <origin xyz="-0.007987 0.262366 -0.985406" rpy="0 0 0"/>
-    <geometry>
-      <mesh filename="package://jaime_description/meshes/l3r_1.stl" scale="0.001 0.001 0.001"/>
-    </geometry>
-  </collision>
-</link>
-<link name="l4r_1">
-  <inertial>
-    <origin xyz="-0.022033052289359936 0.02775238458496604 -0.070094511314298" rpy="0 0 0"/>
-    <mass value="0.1319735958452518"/>
-    <inertia ixx="6.8e-05" iyy="8e-05" izz="7.4e-05" ixy="-0.0" iyz="0.0" ixz="-2e-06"/>
-  </inertial>
-  <visual>
-    <origin xyz="-0.006819 0.290116 -0.815556" rpy="0 0 0"/>
-    <geometry>
-      <mesh filename="package://jaime_description/meshes/l4r_1.stl" scale="0.001 0.001 0.001"/>
-    </geometry>
-    <material name="chassis_material">
-      <color rgba="0.75 0.75 0.75 1.0"/>
-    </material>
-  </visual>
-  <collision>
-    <origin xyz="-0.006819 0.290116 -0.815556" rpy="0 0 0"/>
-    <geometry>
-      <mesh filename="package://jaime_description/meshes/l4r_1.stl" scale="0.001 0.001 0.001"/>
-    </geometry>
-  </collision>
-</link>
-<link name="l5r_1">
-  <inertial>
-    <origin xyz="0.003913819130518236 -6.438555604931784e-05 -0.1904912654580455" rpy="0 0 0"/>
-    <mass value="0.09538513786529154"/>
-    <inertia ixx="0.000748" iyy="0.000753" izz="3e-05" ixy="-0.0" iyz="-0.0" ixz="-5.3e-05"/>
-  </inertial>
-  <visual>
-    <origin xyz="-0.006819 0.262364 -0.767806" rpy="0 0 0"/>
-    <geometry>
-      <mesh filename="package://jaime_description/meshes/l5r_1.stl" scale="0.001 0.001 0.001"/>
-    </geometry>
-    <material name="chassis_material">
-      <color rgba="0.75 0.75 0.75 1.0"/>
-    </material>
-  </visual>
-  <collision>
-    <origin xyz="-0.006819 0.262364 -0.767806" rpy="0 0 0"/>
-    <geometry>
-      <mesh filename="package://jaime_description/meshes/l5r_1.stl" scale="0.001 0.001 0.001"/>
-    </geometry>
-  </collision>
-</link>
-<link name="l6r_1">
-  <inertial>
-    <origin xyz="1.1454308115020628e-07 0.022250384502269127 -0.015076116417858498" rpy="0 0 0"/>
-    <mass value="0.004187419664904639"/>
-    <inertia ixx="2e-06" iyy="1e-06" izz="2e-06" ixy="-0.0" iyz="-0.0" ixz="0.0"/>
-  </inertial>
-  <visual>
-    <origin xyz="-0.007275 0.284614 -0.504262" rpy="0 0 0"/>
-    <geometry>
-      <mesh filename="package://jaime_description/meshes/l6r_1.stl" scale="0.001 0.001 0.001"/>
-    </geometry>
-    <material name="chassis_material">
-      <color rgba="0.75 0.75 0.75 1.0"/>
-    </material>
-  </visual>
-  <collision>
-    <origin xyz="-0.007275 0.284614 -0.504262" rpy="0 0 0"/>
-    <geometry>
-      <mesh filename="package://jaime_description/meshes/l6r_1.stl" scale="0.001 0.001 0.001"/>
-    </geometry>
-  </collision>
-</link>
-<link name="l2h_1">
-  <inertial>
-    <origin xyz="-0.01404344492546073 0.030000481747364617 0.06449858090998739" rpy="0 0 0"/>
-    <mass value="3.4435410806483597"/>
-    <inertia ixx="0.011996" iyy="0.015757" izz="0.017434" ixy="0.0" iyz="-0.0" ixz="-0.000256"/>
-  </inertial>
-  <visual>
-    <origin xyz="-0.007987 0.037366 -1.28382" rpy="0 0 0"/>
-    <geometry>
-      <mesh filename="package://jaime_description/meshes/l2h_1.stl" scale="0.001 0.001 0.001"/>
-    </geometry>
-    <material name="chassis_material">
-      <color rgba="0.75 0.75 0.75 1.0"/>
-    </material>
-  </visual>
-  <collision>
-    <origin xyz="-0.007987 0.037366 -1.28382" rpy="0 0 0"/>
-    <geometry>
-      <mesh filename="package://jaime_description/meshes/l2h_1.stl" scale="0.001 0.001 0.001"/>
-    </geometry>
-  </collision>
-</link>
-<link name="real_sense_1">
-  <inertial>
-    <origin xyz="0.019913541807561386 9.653953529717863e-05 0.02293582384539583" rpy="0 0 0"/>
-    <mass value="0.061254068221964914"/>
-    <inertia ixx="3.4e-05" iyy="1e-05" izz="3.7e-05" ixy="-0.0" iyz="-0.0" ixz="-1e-06"/>
-  </inertial>
-  <visual>
-    <origin xyz="-0.049487 0.007366 -1.40882" rpy="0 0 0"/>
-    <geometry>
-      <mesh filename="package://jaime_description/meshes/real_sense_1.stl" scale="0.001 0.001 0.001"/>
-    </geometry>
-    <material name="chassis_material">
-      <color rgba="0.75 0.75 0.75 1.0"/>
-    </material>
-  </visual>
-  <collision>
-    <origin xyz="-0.049487 0.007366 -1.40882" rpy="0 0 0"/>
-    <geometry>
-      <mesh filename="package://jaime_description/meshes/real_sense_1.stl" scale="0.001 0.001 0.001"/>
-    </geometry>
-  </collision>
-</link>
-<link name="g1r_1">
-  <inertial>
-    <origin xyz="6.478948623842799e-05 3.840721814474257e-07 -0.026736939315767316" rpy="0 0 0"/>
-    <mass value="0.12876405832743776"/>
-    <inertia ixx="8.6e-05" iyy="4.3e-05" izz="7e-05" ixy="-0.0" iyz="-0.0" ixz="0.0"/>
-  </inertial>
-  <visual>
-    <origin xyz="-0.007275 0.262364 -0.480247" rpy="0 0 0"/>
-    <geometry>
-      <mesh filename="package://jaime_description/meshes/g1r_1.stl" scale="0.001 0.001 0.001"/>
-    </geometry>
-    <material name="chassis_material">
-      <color rgba="0.75 0.75 0.75 1.0"/>
-    </material>
-  </visual>
-  <collision>
-    <origin xyz="-0.007275 0.262364 -0.480247" rpy="0 0 0"/>
-    <geometry>
-      <mesh filename="package://jaime_description/meshes/g1r_1.stl" scale="0.001 0.001 0.001"/>
-    </geometry>
-  </collision>
-</link>
-<link name="g2ra_1">
-  <inertial>
-    <origin xyz="-0.0220993118378398 0.01442646877260062 -0.05721188075257794" rpy="0 0 0"/>
-    <mass value="0.05474843522698835"/>
-    <inertia ixx="3.9e-05" iyy="3.7e-05" izz="2e-05" ixy="-0.0" iyz="-1e-05" ixz="0.0"/>
-  </inertial>
-  <visual>
-    <origin xyz="-0.029225 0.243864 -0.438647" rpy="0 0 0"/>
-    <geometry>
-      <mesh filename="package://jaime_description/meshes/g2ra_1.stl" scale="0.001 0.001 0.001"/>
-    </geometry>
-    <material name="chassis_material">
-      <color rgba="0.75 0.75 0.75 1.0"/>
-    </material>
-  </visual>
-  <collision>
-    <origin xyz="-0.029225 0.243864 -0.438647" rpy="0 0 0"/>
-    <geometry>
-      <mesh filename="package://jaime_description/meshes/g2ra_1.stl" scale="0.001 0.001 0.001"/>
-    </geometry>
-  </collision>
-</link>
-<link name="g2rb_1">
-  <inertial>
-    <origin xyz="-0.02210045907599773 -0.014425699768063904 -0.05721188075257849" rpy="0 0 0"/>
-    <mass value="0.05474843522698835"/>
-    <inertia ixx="3.9e-05" iyy="3.7e-05" izz="2e-05" ixy="-0.0" iyz="1e-05" ixz="-0.0"/>
-  </inertial>
-  <visual>
-    <origin xyz="-0.029225 0.280864 -0.438647" rpy="0 0 0"/>
-    <geometry>
-      <mesh filename="package://jaime_description/meshes/g2rb_1.stl" scale="0.001 0.001 0.001"/>
-    </geometry>
-    <material name="chassis_material">
-      <color rgba="0.75 0.75 0.75 1.0"/>
-    </material>
-  </visual>
-  <collision>
-    <origin xyz="-0.029225 0.280864 -0.438647" rpy="0 0 0"/>
-    <geometry>
-      <mesh filename="package://jaime_description/meshes/g2rb_1.stl" scale="0.001 0.001 0.001"/>
-    </geometry>
-  </collision>
-</link>
-<link name="g1l_1">
-  <inertial>
-    <origin xyz="6.478948621099247e-05 -4.2143764839019937e-07 -0.026736939315755603" rpy="0 0 0"/>
-    <mass value="0.12876405832743776"/>
-    <inertia ixx="8.6e-05" iyy="4.3e-05" izz="7e-05" ixy="-0.0" iyz="-0.0" ixz="0.0"/>
-  </inertial>
-  <visual>
-    <origin xyz="-0.007275 -0.247637 -0.480247" rpy="0 0 0"/>
-    <geometry>
-      <mesh filename="package://jaime_description/meshes/g1l_1.stl" scale="0.001 0.001 0.001"/>
-    </geometry>
-    <material name="chassis_material">
-      <color rgba="0.75 0.75 0.75 1.0"/>
-    </material>
-  </visual>
-  <collision>
-    <origin xyz="-0.007275 -0.247637 -0.480247" rpy="0 0 0"/>
-    <geometry>
-      <mesh filename="package://jaime_description/meshes/g1l_1.stl" scale="0.001 0.001 0.001"/>
-    </geometry>
-  </collision>
-</link>
-<link name="g2lb_1">
-  <inertial>
-    <origin xyz="-0.022099311837869458 0.014425663262769728 -0.057211880752566724" rpy="0 0 0"/>
-    <mass value="0.05474843522698835"/>
-    <inertia ixx="3.9e-05" iyy="3.7e-05" izz="2e-05" ixy="-0.0" iyz="-1e-05" ixz="0.0"/>
-  </inertial>
-  <visual>
-    <origin xyz="-0.029225 -0.266137 -0.438647" rpy="0 0 0"/>
-    <geometry>
-      <mesh filename="package://jaime_description/meshes/g2lb_1.stl" scale="0.001 0.001 0.001"/>
-    </geometry>
-    <material name="chassis_material">
-      <color rgba="0.75 0.75 0.75 1.0"/>
-    </material>
-  </visual>
-  <collision>
-    <origin xyz="-0.029225 -0.266137 -0.438647" rpy="0 0 0"/>
-    <geometry>
-      <mesh filename="package://jaime_description/meshes/g2lb_1.stl" scale="0.001 0.001 0.001"/>
-    </geometry>
-  </collision>
-</link>
-<link name="g2la_1">
-  <inertial>
-    <origin xyz="-0.022100459076024488 -0.01442650527789352 -0.057211880752566335" rpy="0 0 0"/>
-    <mass value="0.05474843522698835"/>
-    <inertia ixx="3.9e-05" iyy="3.7e-05" izz="2e-05" ixy="-0.0" iyz="1e-05" ixz="-0.0"/>
-  </inertial>
-  <visual>
-    <origin xyz="-0.029225 -0.229137 -0.438647" rpy="0 0 0"/>
-    <geometry>
-      <mesh filename="package://jaime_description/meshes/g2la_1.stl" scale="0.001 0.001 0.001"/>
-    </geometry>
-    <material name="chassis_material">
-      <color rgba="0.75 0.75 0.75 1.0"/>
-    </material>
-  </visual>
-  <collision>
-    <origin xyz="-0.029225 -0.229137 -0.438647" rpy="0 0 0"/>
-    <geometry>
-      <mesh filename="package://jaime_description/meshes/g2la_1.stl" scale="0.001 0.001 0.001"/>
-    </geometry>
-  </collision>
-</link>
-<link name="laser">
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
Commit message: (MA) navegacion autonoma test

File: jaime_description/urdf/jaime.xacro (robot description, xacro)
@@ -31,3 +31,9 @@
   <origin xyz="0 0 0" rpy="0 0 0"/>
 </joint>
+<link name="laser"/>
+<joint name="laser_joint" type="fixed">
+  <parent link="base_link"/>
+  <child link="laser"/>
+  <origin xyz="0 0 0" rpy="0 0 ${-pi}"/>
+</joint>
 </robot>
