Commit message: Update jaime realsense urdf

File: jaime_description/robots/jaime_realsense.urdf.xacro (robot description, xacro)
@@ -12,5 +12,5 @@
   <sensor_d435 parent="link_palo">
     <!--origin xyz="0.0 0.0 0" rpy="0 ${-M_PI/3} 0"/-->
-    <origin xyz="0.1 0.0 0.0" rpy="0 ${M_PI/4} 0"/>
+    <origin xyz="0.08 0.0 0.0" rpy="0 0.785398 0"/>
 	</sensor_d435>
   <kobuki/>

File: jaime_description/urdf/jaime_realsense.urdf.xacro (robot description, xacro)
@@ -289,5 +289,5 @@
       <visual>
         <geometry>
-          <mesh filename="package://jaime_description/meshes/kobuki_hospital.stl"/>
+          <mesh filename="package://jaime_description/meshes/test_DR.stl"/>
         </geometry>
         <origin xyz="0 0 0" rpy="0 0 ${M_PI/2}"/>
@@ -295,5 +295,5 @@
     </link>
     <joint name="case_to_base_link" type="fixed">
-      <origin xyz="0 0 0.12"/>
+      <origin xyz="0 0 0"/>
       <parent link="base_link"/>
       <child link="case"/>

Commit message: add laser_link

File: jaime_description/robots/jaime_realsense.urdf.xacro (robot description, xacro)
@@ -10,7 +10,7 @@
   <xacro:include filename="$(find realsense2_description)/urdf/_d435.urdf.xacro"/>
   <xacro:property name="M_PI" value="3.1415926535897931" />
-  <sensor_d435 parent="link_palo">
+  <sensor_d435 parent="laser_link">
     <!--origin xyz="0.0 0.0 0" rpy="0 ${-M_PI/3} 0"/-->
-    <origin xyz="0.08 0.0 0.0" rpy="0 0.785398 0"/>
+    <origin xyz="0.0 0.0 0.0" rpy="0 ${-M_PI/5} 0"/>
 	</sensor_d435>
   <kobuki/>

File: jaime_description/urdf/jaime_realsense.urdf.xacro (robot description, xacro)
@@ -257,6 +257,11 @@
     <!---->
     <link name="camara_profundidad" type="fixed"/>
-    <link name="link_palo" type="fixed">
-    </link>
+    <link name="link_palo" type="fixed"/>
+    <link name="laser_link" type="fixed"/>
+    <joint name="base_link_to_laser_link" type="fixed">
+      <origin xyz="0.15 0.0 0.13"/>
+      <parent link="base_link"/>
+      <child link="laser_link"/>
+    </joint>
     <!--joint name="link_palo_base" type="fixed"-->
     <joint name="link_palo_to_pc_base_up" type="fixed">

Commit message: Clean pudu urdf and change camera position

File: jaime_description/robots/jaime_realsense.urdf.xacro (robot description, xacro)
@@ -8,9 +8,9 @@
   <xacro:include filename="$(find jaime_description)/urdf/jaime_realsense.urdf.xacro" />
   <!-- Add Realsense -->
-  <xacro:include filename="$(find realsense2_description)/urdf/_d435.urdf.xacro"/>
+  <xacro:include filename="$(find uchile_sensors)/urdf/_d435.urdf.xacro"/>
   <xacro:property name="M_PI" value="3.1415926535897931" />
   <sensor_d435 parent="laser_link">
     <!--origin xyz="0.0 0.0 0" rpy="0 ${-M_PI/3} 0"/-->
-    <origin xyz="0.0 0.0 0.0" rpy="0 ${-M_PI/5} 0"/>
+    <origin xyz="0.0 0.0 0.0" rpy="${M_PI/2} 0.47 0"/>
 	</sensor_d435>
   <kobuki/>

File: jaime_description/urdf/jaime_realsense.urdf.xacro (robot description, xacro)
@@ -212,82 +212,9 @@
       </inertial>
     </link>
-    <!-- kobuki agrega link_palo y base-->
-    <joint name="camara_joint" type="fixed">
-      <axis xyz="0 1 0" />
-      <origin xyz="0 0 0.8" rpy="0 0 0"/>
-      <parent link="link_palo"/>
-      <child link="camara"/>
-    </joint>
-    <!--joint camara de profunidad-->
-    <joint name="camara_profundidad_joint" type="fixed">
-      <!--axis xyz="0 1 0" /-->
-      <origin xyz ="0.1 0 0.15" rpy="0 0 0"/>  <!--heght480-640/2-->
-      <!--parent link="base_link"/-->
-      <parent link="pc_base_up"/>
-      <child link="camara_profundidad"/>
-    </joint>
-    <joint name="camara_profundidad_optical_joint" type="fixed">
-  <origin xyz="0 0 0" rpy="${-M_PI/2} 0 ${-M_PI/2}" />
-  <parent link="camara_profundidad" />
-  <child link="camara_profundidad_optical" />
-</joint>
-<link name="camara_profundidad_optical"/>
-    <link name="camara">
-      <!--collision>
-        <origin xyz="0 0 0" rpy="0 0 0"/>
-        <geometry>
-      <box size="${camara ${camara} ${camara}"/>
-        </geometry>
-      </collision-->
-      <visual>
-        <origin xyz="0 0 0" rpy="${M_PI/2} ${M_PI/2} ${M_PI/2}"/>
-        <geometry>
-          <!--box size="${camara} ${camara} ${camara}"/-->
-          <mesh filename="package://jaime_description/meshes/camera_ASUS_XTION.STL"/>
-        </geometry>
-        <material name="red"/>
-      </visual>
-      <!--inertial>
-        <mass value="1e-5" />
-        <origin xyz="0 0 0" rpy="0 0 0"/>
-        <inertia ixx="1e-6" ixy="0" ixz="0" iyy="1e-6" iyz="0" izz="1e-6" />
-      </inertial-->
-    </link>
-    <!--camara de profunidad, kinetic microsoft-->
-    <!---->
-    <link name="camara_profundidad" type="fixed"/>
-    <link name="link_palo" type="fixed"/>
     <link name="laser_link" type="fixed"/>
     <joint name="base_link_to_laser_link" type="fixed">
-      <origin xyz="0.15 0.0 0.13"/>
+      <origin xyz="0.0861 0.0125 0.935"/>
       <parent link="base_link"/>
       <child link="laser_link"/>
-    </joint>
-    <!--joint name="link_palo_base" type="fixed"-->
-    <joint name="link_palo_to_pc_base_up" type="fixed">
-      <origin xyz="0 0 0.8"/>
-      <parent link="pc_base_up"/>
-      <child link="link_palo"/>
-    </joint>
-    <link name="pc_base_down" type="fixed">
-    </link>
-    <joint name="pc_base_down_to_base_link" type="fixed">
-      <origin xyz="0 0 0.1"/>
-      <parent link="base_link"/>
-      <child link="pc_base_down"/>
-    </joint>
-    <link name="pc_base_up" type="fixed">
-    </link>
-    <joint name="pc_base_up_to_base_link" type="fixed">
-      <origin xyz="0 0 0.18"/>
-      <parent link="base_link"/>
-      <child link="pc_base_up"/>
-    </joint>
-    <link name="wood_base" type="fixed">
-    </link>
-    <joint name="wood_base_to_base_link" type="fixed">
-      <origin xyz="0 0 -0.018"/>
-      <parent link="base_link"/>
-      <child link="wood_base"/>
     </joint>
     <link name="case" type="fixed">
@@ -304,7 +231,7 @@
       <child link="case"/>
     </joint>
-    <!-- Kobuki Gazebo simulation details -->
-    <kobuki_sim/>
-  </xacro:macro>
+<!-- Kobuki Gazebo simulation details -->
+<kobuki_sim/>
+</xacro:macro>
 </robot>
 </world>

File: jaime_description/urdf/jaime_realsense_gazebo.urdf.xacro (robot description, xacro)
@@ -46,45 +46,4 @@
 	    </sensor>
 	  </gazebo>
-    <gazebo reference="link_palo">
-      <material>Gazebo/Black</material>
-    </gazebo>
-    <!-- camara rql-->
-    <gazebo reference="camara">
-      <material>Gazebo/Black</material>
-      <sensor type="camera" name="camara_1">
-        <update_rate>30</update_rate>
-        <camera name="head">
-          <horizontal_fov>1.396234</horizontal_fov>
-          <image>
-            <width>800</width>
-            <height>800</height>
-            <format>R8G8B8</format>
-          </image>
-          <clip>
-            <near>0.02</near>
-            <far>300</far>
-          </clip>
-          <noise>
-            <type>gaussian</type>
-            <mean>0.0</mean>
-            <stddev>0.007</stddev>
-          </noise>
-        </camera>
-        <plugin name="camera_controller" filename="libgazebo_ros_camera.so">
-          <alwaysOn>true</alwaysOn>
-          <updateRate>0.0</updateRate>
-          <cameraName>kobuki_sim/camera_1</cameraName>
-          <imageTopicName>image_raw</imageTopicName>
-          <cameraInfoTopicName>camera_info</cameraInfoTopicName>
-          <frameName>camara</frameName>
-          <hackBaseline>0.07</hackBaseline>
-          <distortionK1>0.0</distortionK1>
-          <distortionK2>0.0</distortionK2>
-          <distortionK3>0.0</distortionK3>
-          <distortionT1>0.0</distortionT1>
-          <distortionT2>0.0</distortionT2>
-        </plugin>
-      </sensor>
-    </gazebo>
 	  <gazebo reference="cliff_sensor_left_link">
 	    <sensor type="ray" name="cliff_sensor_left">
