Commit message: (MA) editado jaime xacro, ahora display se ve normal fuera de docker

File: src/jaime_description/urdf/jaime.xacro (robot description, xacro)
@@ -177,9 +177,10 @@
 </joint>
 <joint name="odom_to_base_link" type="floating">
+  <origin xyz= "0.0 0.0 0.0" rpy="0 0 0"/>
   <parent link="odom"/>
   <child link="base_link"/>
 </joint>
 <joint name="kobuki_base_joint" type="fixed">
-  <origin xyz="0 0 0.1" rpy="0 0 0" />
+  <origin xyz="0 0 -0.1" rpy="0 0 0" />
   <parent link="base_link"/>
   <child link="kobuki_base_link" />

File: src/jaime_description/urdf/kobuki_urdf.xacro (robot description, xacro)
@@ -10,5 +10,5 @@
   <!-- Kobuki -->
   <xacro:macro name="kobuki" params = "namespace">
-    <link name="${namespace}base_link"> #ver si se puede subir desde aca
+    <link name="${namespace}base_link">
       <visual>
         <geometry>

Commit message: (MA) arreglado problema de display_launch

File: src/jaime_description/urdf/jaime.xacro (robot description, xacro)
@@ -165,11 +165,11 @@
   </collision>
 </link>
-<link name="world">
-</link>
-<link name="odom"/>
+<!-- <link name="world">
+</link>
+<link name="odom"/> -->
 <!-- ver porque estan los dos de nuevo-->
 <!-- inicio joints -->
 <!-- se conecto kobuki a base_link y todo lo demas se conecto a kobuki despues -->
-<joint name="world_to_odom" type="fixed">
+<!-- <joint name="world_to_odom" type="fixed">
   <origin xyz="0.0 0.0 0.0" rpy="0 0 0"/>
   <parent link="world"/>
@@ -180,5 +180,5 @@
   <parent link="odom"/>
   <child link="base_link"/>
-</joint>
+</joint> -->
 <joint name="kobuki_base_joint" type="fixed">
   <origin xyz="0 0 -0.1" rpy="0 0 0" />
